File: motor-driver/inverter.kicad_sch (KiCad schematic)
At the start: 24 parts, among them Q10 NMOS, Q11 NMOS, Q12 NMOS, Q7 NMOS, Q8 NMOS, Q9 NMOS

Commit message: added connectors starting pcb layout
Parts:
- C8: footprint Capacitor_SMD:C_0201_0603Metric_Pad0.64x0.40mm_HandSolder -> 330uFCap:CAPPRD500W60D1000H1400
- Q10, Q11, Q12, Q7, Q8, Q9: footprint (none) -> IPD090N03L:DPAK228P998X235-3N
- R26, R27, R28, R30, R31, R32, R33, R35, R36, R55, R56, R6: footprint (none) -> Resistor_SMD:R_0805_2012Metric
- R29, R34, R57: footprint (none) -> Resistor_SMD:R_2512_6332Metric
Other:
- note added: "1 electrolytic (330uF), 2 ceramic (47uF, 1uF)"
- note added: "MOTOR BULK CAPACITORS"
Changed lines of the file:
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@@
 	(generator_version "9.0")
 	(paper "A4")
+	(text "MOTOR BULK CAPACITORS"
+		(exclude_from_sim no)
+		(at 221.234 19.05 0)
+		(effects
+			(font
+				(size 2.54 2.54)
+			)
+		)
+	)
+	(text "1 electrolytic (330uF), 2 ceramic (47uF, 1uF)"
+		(exclude_from_sim no)
+		(at 239.776 45.466 0)
+		(effects
+			(font
+				(size 1.27 1.27)
+			)
+		)
+	)
 	(junction
 		(at 135.89 129.54)
@@
 			(width 0)
 			(type default)
-		)
-	)
-	(label "MOTOR BULK CAPACITORS"
-		(at 198.12 20.32 0)
-		(effects
-			(font
-				(size 2.54 2.54)
-				(thickness 0.254)
-				(bold yes)
-			)
-			(justify left bottom)
-		)
-	)
-	(label "1 electrolytic (330uF), 2 ceramic (47uF, 1uF)"
-		(at 215.9 40.64 0)
-		(effects
-			(font
-				(size 1.27 1.27)
-			)
-			(justify left bottom)
 		)
 	)
@@
 			)
 		)
-		(property "Footprint" ""
+		(property "Footprint" "IPD090N03L:DPAK228P998X235-3N"
 			(at 93.98 72.39 0)
 			(effects
@@
 			)
 		)
-		(property "Footprint" ""
+		(property "Footprint" "IPD090N03L:DPAK228P998X235-3N"
 			(at 257.81 73.66 0)
 			(effects
@@
 			)
 		)
-		(property "Footprint" ""
+		(property "Footprint" "Resistor_SMD:R_0805_2012Metric"
 			(at 240.03 105.918 90)
 			(effects
@@
 			)
 		)
-		(property "Footprint" ""
+		(property "Footprint" "Resistor_SMD:R_0805_2012Metric"
 			(at 69.85 105.918 90)
 			(effects
@@
 			)
 		)
-		(property "Footprint" ""
+		(property "Footprint" "Resistor_SMD:R_0805_2012Metric"
 			(at 50.038 96.52 90)
 			(effects
@@
 			)
 		)
-		(property "Footprint" ""
+		(property "Footprint" "Resistor_SMD:R_0805_2012Metric"
 			(at 129.54 76.708 90)
 			(effects
@@
 			)
 		)
-		(property "Footprint" ""
+		(property "Footprint" "Resistor_SMD:R_0805_2012Metric"
 			(at 137.668 95.25 90)
 			(effects
@@
 			)
 		)
-		(property "Footprint" ""
+		(property "Footprint" "Resistor_SMD:R_0805_2012Metric"
 			(at 215.138 104.14 90)
 			(effects
@@
 			)
 		)
-		(property "Footprint" ""
+		(property "Footprint" "IPD090N03L:DPAK228P998X235-3N"
 			(at 175.26 72.39 0)
 			(effects
@@
 			)
 		)
-		(property "Footprint" ""
+		(property "Footprint" "Resistor_SMD:R_0805_2012Metric"
 			(at 165.608 115.57 90)
 			(effects
@@
 			)
 		)
-		(property "Footprint" ""
+		(property "Footprint" "IPD090N03L:DPAK228P998X235-3N"
 			(at 257.81 101.6 0)
 			(effects
@@
 			)
 		)
-		(property "Footprint" ""
+		(property "Footprint" "Resistor_SMD:R_0805_2012Metric"
 			(at 160.02 105.918 90)
 			(effects
@@
 			)
 		)
-		(property "Footprint" ""
+		(property "Footprint" "Resistor_SMD:R_2512_6332Metric"
 			(at 93.218 120.65 90)
 			(effects
@@
 			)
 		)
-		(property "Footprint" ""
+		(property "Footprint" "Resistor_SMD:R_0805_2012Metric"
 			(at 207.01 77.978 90)
 			(effects
@@
 			)
 		)
-		(property "Footprint" ""
+		(property "Footprint" "IPD090N03L:DPAK228P998X235-3N"
 			(at 93.98 101.6 0)
 			(effects
@@
 			)
 		)
-		(property "Footprint" ""
+		(property "Footprint" "Resistor_SMD:R_0805_2012Metric"
 			(at 246.888 116.84 90)
 			(effects
@@
 			)
 		)
-		(property "Footprint" ""
+		(property "Footprint" "Resistor_SMD:R_0805_2012Metric"
 			(at 80.518 116.84 90)
 			(effects
@@
 			)
 		)
-		(property "Footprint" "Capacitor_SMD:C_0201_0603Metric_Pad0.64x0.40mm_HandSolder"
+		(property "Footprint" "330uFCap:CAPPRD500W60D1000H1400"
 			(at 209.2452 34.29 0)
 			(effects
@@
 			)
 		)
-		(property "Footprint" ""
+		(property "Footprint" "Resistor_SMD:R_0805_2012Metric"
 			(at 38.1 76.708 90)
 			(effects
@@
 			)
 		)
-		(property "Footprint" ""
+		(property "Footprint" "Resistor_SMD:R_2512_6332Metric"
 			(at 174.498 121.92 90)
 			(effects
@@
 			)
 		)
-		(property "Footprint" ""
+		(property "Footprint" "Resistor_SMD:R_2512_6332Metric"
 			(at 257.048 123.19 90)
 			(effects
@@
 			)
 		)
-		(property "Footprint" ""
+		(property "Footprint" "IPD090N03L:DPAK228P998X235-3N"
 			(at 175.26 101.6 0)
 			(effects

Commit message: commit before changing custom sullen key sense
Parts:
- removed C8: 330uF, 330uFCap:CAPPRD500W60D1000H1400, symbol Device:C
- removed Q10, Q11, Q12, Q7, Q8, Q9: NMOS, IPD090N03L:DPAK228P998X235-3N, symbol Simulation_SPICE:NMOS
- added C1, C44, C45, C46, C47, C48, C49, C50, C51, C52: 10uF, Capacitor_SMD:C_0603_1608Metric, symbol Device:C
- added C42: 330uF, A768MS337M1VLAS022:CAPAE1030X1225N, symbol A768MS337M1VLAS022:A768MS337M1VLAS022
- added MOSFET1, MOSFET2, MOSFET3, MOSFET4, MOSFET5, MOSFET6: AON6512, AON6512:DFN5X6_8L_EP1_P_AOS, symbol AON6512:AON6512
- C14: value 47uF -> 10uF; footprint Capacitor_SMD:C_0201_0603Metric_Pad0.64x0.40mm_HandSolder -> Capacitor_SMD:C_0603_1608Metric
- C15: value 1uF -> 10uF; footprint Capacitor_SMD:C_0201_0603Metric_Pad0.64x0.40mm_HandSolder -> Capacitor_SMD:C_0603_1608Metric
- R26, R27, R28, R30, R31, R32, R33, R35, R36, R55, R56, R6: footprint Resistor_SMD:R_0805_2012Metric -> Resistor_SMD:R_0603_1608Metric
Connections:
- net MOTOR_GND: now also C1.2, C42.2, C44.2, C45.2, C46.2, C47.2, C48.2, C49.2, C50.2, C51.2, C52.2
- net U_LEG_BST: now also MOSFET1.1, MOSFET1.2, MOSFET1.3, MOSFET2.5, MOSFET2.6, MOSFET2.7, MOSFET2.8
- net U_SENSE: now also MOSFET2.1, MOSFET2.2, MOSFET2.3
- net V_BUS: now also C1.1, C42.1, C44.1, C45.1, C46.1, C47.1, C48.1, C49.1, C50.1, C51.1, C52.1, MOSFET1.5, MOSFET1.6, MOSFET1.7, MOSFET1.8, MOSFET3.5, MOSFET3.6, MOSFET3.7, MOSFET3.8, MOSFET4.5, MOSFET4.6, MOSFET4.7, MOSFET4.8
- net V_LEG_BST: now also MOSFET3.1, MOSFET3.2, MOSFET3.3, MOSFET5.5, MOSFET5.6, MOSFET5.7, MOSFET5.8
- net V_SENSE: now also MOSFET5.1, MOSFET5.2, MOSFET5.3
- net W_LEG_BST: now also MOSFET4.1, MOSFET4.2, MOSFET4.3, MOSFET6.5, MOSFET6.6, MOSFET6.7, MOSFET6.8
- net W_SENSE: now also MOSFET6.1, MOSFET6.2, MOSFET6.3
- net at R26.2, R28.2: now also MOSFET1.4
- net at R36.2, R56.2: now also MOSFET4.4
- net at R35.2, R55.2: now also MOSFET6.4
- net at R27.2, R6.2: now also MOSFET2.4
- net at R31.2, R33.2: now also MOSFET3.4
- net at R30.2, R32.2: now also MOSFET5.4
Other:
- note added: "Aluminum Polymer bus 330uF further away, ceramic bus 4 x 10uF near each inverter"
- note removed: "1 electrolytic (330uF), 2 ceramic (47uF, 1uF)"
- moved on the sheet: R26, R27, R28, R29, R30, R31, R32, R33, R34, R35, R36, R55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

Commit message: commit before inverter revisions
Parts:
- added U: U_PAD, symbol Connector:TestPoint
- added V: V_PAD, symbol Connector:TestPoint
- added W: W_PAD, symbol Connector:TestPoint
Connections:
- net MOTOR_GND: now also MOSFET2.1, MOSFET2.2, MOSFET2.3, MOSFET5.1, MOSFET5.2, MOSFET5.3, MOSFET6.1, MOSFET6.2, MOSFET6.3; no longer R29.1, R34.1, R57.1
- net U_LEG_BST: now also R29.2
- net V_LEG_BST: now also R34.2
- net W_LEG_BST: now also R57.2
- removed net U_SENSE: MOSFET2.1, MOSFET2.2, MOSFET2.3, R29.2
- removed net V_SENSE: MOSFET5.1, MOSFET5.2, MOSFET5.3, R34.2
- removed net W_SENSE: MOSFET6.1, MOSFET6.2, MOSFET6.3, R57.2
- new net U_BACK_EMF: R29.1, U.1
- new net V_SENSE-: R34.1, V.1
- new net W_SENSE-: R57.1, W.1
Other:
- moved on the sheet: C42, MOSFET2, MOSFET5, MOSFET6, R27, R28, R30, R32, R35, R55, R6

Commit message: post revisions
Parts:
- removed C1, C14, C15, C44, C45, C46, C47, C48, C49, C50, C51, C52: 10uF, Capacitor_SMD:C_0603_1608Metric, symbol Device:C
- removed MOSFET1, MOSFET2, MOSFET3, MOSFET4, MOSFET5, MOSFET6: AON6512, AON6512:DFN5X6_8L_EP1_P_AOS, symbol AON6512:AON6512
- removed R26, R27, R31, R32, R36, R55: 22, Resistor_SMD:R_0603_1608Metric, symbol Device:R
- removed R28, R30, R33, R35, R56, R6: 10k, Resistor_SMD:R_0603_1608Metric, symbol Device:R
- removed R29, R34, R57: 5m, Resistor_SMD:R_2512_6332Metric, symbol Device:R
- removed U: U_PAD, symbol Connector:TestPoint
- removed V: V_PAD, symbol Connector:TestPoint
- removed W: W_PAD, symbol Connector:TestPoint
- added R95, R96, R97: 10k, Resistor_SMD:R_0603_1608Metric, symbol Device:R
Connections:
- net MOTOR_GND renamed GND
- new net MOTOR_NEUTRAL_REF: R95.2, R96.2, R97.2
- new net back_emf_u/BEMF: R95.1
- new net back_emf_v/BEMF: R96.1
- new net back_emf_w/BEMF: R97.1
Other:
- added sheet back_emf_u (back_emf.kicad_sch)
- added sheet back_emf_v (back_emf.kicad_sch)
- added sheet back_emf_w (back_emf.kicad_sch)
- added sheet current_sense_u (current_sense.kicad_sch)
- added sheet current_sense_v (current_sense.kicad_sch)
- added sheet current_sense_w (current_sense.kicad_sch)
- added sheet gate-driver (gate-driver.kicad_sch)
- added sheet inverter_u (inverter_leg.kicad_sch)
- added sheet inverter_v (inverter_leg.kicad_sch)
- added sheet inverter_w (inverter_leg.kicad_sch)
- note added: "Aluminum Bulk Capacitor"
- note added: "Aluminum Polymer. Additional Ceramic buses are close to legs Can be further from legs than ceramics"
- note added: "Back EMF Sensing"
- note added: "Current Sensing"
- note added: "Gate Driver"
- note added: "Inverter Legs"
- note removed: "Aluminum Polymer bus 330uF further away, ceramic bus 4 x 10uF near each inverter"
- note removed: "MOTOR BULK CAPACITORS"
- company: (none) -> Drone 
- moved on the sheet: C42

Commit message: added spi connection
Parts:
- added NEUTRAL1: TestPoint, TestPoint:TestPoint_Loop_D1.80mm_Drill1.0mm_Beaded, symbol Connector:TestPoint
Connections:
- net MOTOR_NEUTRAL_REF: now also NEUTRAL1.1
Changed lines of the file:
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@@
 		(color 0 0 0 0)
 	)
+	(junction
+		(at 240.03 40.64)
+		(diameter 0)
+		(color 0 0 0 0)
+	)
 	(wire
 		(pts
@@
 	(wire
 		(pts
+			(xy 240.03 40.64) (xy 242.57 40.64)
+		)
+		(stroke
+			(width 0)
+			(type default)
+		)
+	)
+	(wire
+		(pts
 			(xy 26.67 68.58) (xy 30.48 68.58)
 		)
@@
 	(wire
 		(pts
-			(xy 237.49 40.64) (xy 242.57 40.64)
+			(xy 237.49 40.64) (xy 240.03 40.64)
 		)
 		(stroke
@@
 					(unit 1)
 				)
+			)
+		)
+	)
+	(symbol
+		(lib_id "Connector:TestPoint")
+		(at 240.03 40.64 180)
+		(unit 1)
+		(exclude_from_sim no)
+		(in_bom no)
+		(on_board yes)
+		(dnp no)
+		(fields_autoplaced yes)
+		(property "Reference" "NEUTRAL1"
+			(at 242.57 42.6719 0)
+			(effects
+				(font
+					(size 1.27 1.27)
+				)
+				(justify right)
+			)
+		)
+		(property "Value" "TestPoint"
+			(at 242.57 45.2119 0)
+			(effects
+				(font
+					(size 1.27 1.27)
+				)
+				(justify right)
+			)
+		)
+		(property "Footprint" "TestPoint:TestPoint_Loop_D1.80mm_Drill1.0mm_Beaded"
+			(at 234.95 40.64 0)
+			(effects
+				(font
+					(size 1.27 1.27)
+				)
+				(hide yes)
+			)
+		)
+		(property "Datasheet" "~"
+			(at 234.95 40.64 0)
+			(effects
+				(font
+					(size 1.27 1.27)
+				)
+				(hide yes)
+			)
+		)
+		(property "Description" "test point"
+			(at 240.03 40.64 0)
+			(effects
+				(font
+					(size 1.27 1.27)
+				)
+				(hide yes)
+			)
+		)
+		(pin "1"
+		)
+		(instances
+			(project "motor-driver"
+				(path "/2980fc7e-b297-4843-ba9f-cceafa384b2f/d36b7053-ee22-4492-bdec-8a6a56460e2b"
+					(reference "NEUTRAL1")
+					(unit 1)
+				)

Commit message: added test points
Parts:
- removed NEUTRAL1: TestPoint, TestPoint:TestPoint_Loop_D1.80mm_Drill1.0mm_Beaded, symbol Connector:TestPoint
- added BEMFU1, NEUTRAL, SENSEW1, WGATE_BST1, WGATE_H1: TestPoint, TestPoint:TestPoint_THTPad_D1.0mm_Drill0.5mm, symbol Connector:TestPoint
Connections:
- net BEMF_U: now also BEMFU1.1
- net CURRENT_SENSE_W: now also SENSEW1.1
- net MOTOR_NEUTRAL_REF: now also NEUTRAL.1
- net gate-driver/W_GATE_H: now also WGATE_H1.1
- net gate-driver/W_LEG_BST: now also WGATE_BST1.1

Commit message: bom finished
Parts:
- C42: value 330uF -> 330u; Availability In Stock -> (none); CREATOR AAMIR -> (none); Check_prices https://www.snapeda.com/parts/A768MS337M1VLAS022/Kemet/view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 -> (none); Description_1 330 µF 35 V Aluminum - Polymer Capacitors Radial, Can - SMD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 -> (none); MPN (none) -> A768MS337M1VLAS022; Supplier (none) -> Digikey
- R95, R96, R97: MANUFACTURER (none) -> YAGEO; MPN (none) -> RC0603FR-0710KL; Supplier (none) -> Digikey
- renumbered NEUTRAL to NEUTRAL1
Changed lines of the file:
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@@
 		(on_board yes)
 		(dnp no)
-		(property "Reference" "NEUTRAL"
+		(property "Reference" "NEUTRAL1"
 			(at 244.094 45.974 0)
 			(effects
@@
 		)
 		(property "Description" "test point"
+			(at 240.03 40.64 0)
+			(effects
+				(font
+					(size 1.27 1.27)
+				)
+				(hide yes)
+			)
+		)
+		(property "MPN" ""
+			(at 240.03 40.64 0)
+			(effects
+				(font
+					(size 1.27 1.27)
+				)
+				(hide yes)
+			)
+		)
+		(property "Supplier" ""
 			(at 240.03 40.64 0)
 			(effects
@@
 			(project "motor-driver"
 				(path "/2980fc7e-b297-4843-ba9f-cceafa384b2f/d36b7053-ee22-4492-bdec-8a6a56460e2b"
-					(reference "NEUTRAL")
+					(reference "NEUTRAL1")
 					(unit 1)
 				)
@@
 		)
 		(property "Description" "test point"
+			(at 90.17 139.7 0)
+			(effects
+				(font
+					(size 1.27 1.27)
+				)
+				(hide yes)
+			)
+		)
+		(property "MPN" ""
+			(at 90.17 139.7 0)
+			(effects
+				(font
+					(size 1.27 1.27)
+				)
+				(hide yes)
+			)
+		)
+		(property "Supplier" ""
 			(at 90.17 139.7 0)
 			(effects
@@
 			)
 		)
+		(property "MPN" "RC0603FR-0710KL"
+			(at 227.33 30.48 90)
+			(effects
+				(font
+					(size 1.27 1.27)
+				)
+				(hide yes)
+			)
+		)
+		(property "Supplier" "Digikey"
+			(at 227.33 30.48 90)
+			(effects
+				(font
+					(size 1.27 1.27)
+				)
+				(hide yes)
+			)
+		)
+		(property "MANUFACTURER" "YAGEO"
+			(at 227.33 30.48 90)
+			(effects
+				(font
+					(size 1.27 1.27)
+				)
+				(hide yes)
+			)
+		)
 		(pin "2"
 		)
@@
 			)
 		)
+		(property "MPN" "RC0603FR-0710KL"
+			(at 227.33 40.64 90)
+			(effects
+				(font
+					(size 1.27 1.27)
+				)
+				(hide yes)
+			)
+		)
+		(property "Supplier" "Digikey"
+			(at 227.33 40.64 90)
+			(effects
+				(font
+					(size 1.27 1.27)
+				)
+				(hide yes)
+			)
+		)
+		(property "MANUFACTURER" "YAGEO"
+			(at 227.33 40.64 90)
+			(effects
+				(font
+					(size 1.27 1.27)
+				)
+				(hide yes)
+			)
+		)
 		(pin "2"
 		)
@@
 			)
 		)
-		(property "Value" "330uF"
+		(property "Value" "330u"
 			(at 160.02 169.6065 90)
 			(effects
@@
 			)
 		)
-		(property "CREATOR" "AAMIR"
-			(at 156.21 167.64 0)
-			(effects
-				(font
-					(size 1.27 1.27)
-				)
-				(justify bottom)
-				(hide yes)
-			)
-		)
 		(property "Price" "None"
 			(at 156.21 167.64 0)
@@
 			)
 		)
-		(property "Check_prices" "https://www.snapeda.com/parts/A768MS337M1VLAS022/Kemet/view-part/?ref=eda"
-			(at 156.21 167.64 0)
-			(effects
-				(font
-					(size 1.27 1.27)
-				)
-				(justify bottom)
-				(hide yes)
-			)
-		)
 		(property "STANDARD" "IPC-7351B"
 			(at 156.21 167.64 0)
@@
 			)
 		)
-		(property "Description_1" "330 µF 35 V Aluminum - Polymer Capacitors Radial, Can - SMD 22mOhm 2000 Hrs @ 125°C"
-			(at 156.21 167.64 0)
-			(effects
-				(font
-					(size 1.27 1.27)
-				)
-				(justify bottom)
-				(hide yes)
-			)
-		)
-		(property "Availability" "In Stock"
-			(at 156.21 167.64 0)
-			(effects
-				(font
-					(size 1.27 1.27)
-				)
-				(justify bottom)
-				(hide yes)
-			)
-		)
 		(property "MANUFACTURER" "KEMET"
 			(at 156.21 167.64 0)
@@
 				)
 				(justify bottom)
+				(hide yes)
+			)
+		)
+		(property "MPN" "A768MS337M1VLAS022"
+			(at 156.21 167.64 90)
+			(effects
+				(font
+					(size 1.27 1.27)
+				)
+				(hide yes)
+			)
+		)
+		(property "Supplier" "Digikey"
+			(at 156.21 167.64 90)
+			(effects
+				(font
+					(size 1.27 1.27)
+				)
 				(hide yes)
 			)
@@
 			)
 		)
+		(property "MPN" ""
+			(at 104.14 124.46 0)
+			(effects
+				(font
+					(size 1.27 1.27)
+				)
+				(hide yes)
+			)
+		)
+		(property "Supplier" ""
+			(at 104.14 124.46 0)
+			(effects
+				(font
+					(size 1.27 1.27)
+				)
+				(hide yes)
+			)
+		)
 		(pin "1"
 		)
@@
 			)
 		)
+		(property "MPN" ""
+			(at 248.8459 69.85 0)
+			(effects
+				(font
+					(size 1.27 1.27)
+				)
+				(hide yes)
+			)
+		)
+		(property "Supplier" ""
+			(at 248.8459 69.85 0)
+			(effects
+				(font
+					(size 1.27 1.27)
+				)
+				(hide yes)
+			)
+		)
 		(pin "1"
 		)
@@
 		)
 		(property "Description" "test point"
+			(at 93.98 142.24 0)
+			(effects
+				(font
+					(size 1.27 1.27)
+				)
+				(hide yes)
+			)
+		)
+		(property "MPN" ""
+			(at 93.98 142.24 0)
+			(effects
+				(font
+					(size 1.27 1.27)
+				)
+				(hide yes)
+			)
+		)
+		(property "Supplier" ""
 			(at 93.98 142.24 0)
 			(effects
@@
 			(effects
 				(font
+					(size 1.27 1.27)
+				)
+				(hide yes)
+			)
+		)
+		(property "MPN" "RC0603FR-0710KL"
+			(at 227.33 52.07 90)
+			(effects
+				(font
+					(size 1.27 1.27)
+				)
+				(hide yes)
+			)
+		)
+		(property "Supplier" "Digikey"
+			(at 227.33 52.07 90)
+			(effects
+				(font
+					(size 1.27 1.27)
+				)
+				(hide yes)
+			)
+		)
+		(property "MANUFACTURER" "YAGEO"
+			(at 227.33 52.07 90)
+			(effects
+				(font
