File: motor-driver/motor-driver.kicad_sch (KiCad schematic)
At the start: 0 parts

Commit message: added test points
Parts:
- added 3V3, 5V1, GND1, VBUS1: TestPoint, TestPoint:TestPoint_THTPad_D1.0mm_Drill0.5mm, symbol Connector:TestPoint
Connections:
- new net 3V3: 3V3.1
- new net 5V: 5V1.1
- new net GND: GND1.1
- new net V_BUS: VBUS1.1
Other:
- note added: "Power Test Points"
