File: motor-driver/inverter_leg.kicad_sch (KiCad schematic)
At the start: 15 parts

Commit message: routing complete
Parts:
- removed NT1, NT4, NT7: net-tie, symbol Device:NetTie_3_Tee
- V1: renamed from MOTOR_CONNECT2; footprint (none) -> TestPoint:TestPoint_Pad_4.0x4.0mm
Connections:
- net SHUNT_N is gone; now on net BACK_EMF: V1.1
- net SHUNT_P is gone; now on net BST: MOSFET8.5, MOSFET8.6, MOSFET8.7, MOSFET8.8
- net BACK_EMF: now also R70.1
- net BST: now also MOSFET7.1, MOSFET7.2, MOSFET7.3, R70.2

Commit message: added spi connection
Parts:
- added GATE_H2, GATE_L2, SHUNT+2, SHUNT-2: TestPoint, TestPoint:TestPoint_Loop_D1.80mm_Drill1.0mm_Beaded, symbol Connector:TestPoint
- C43, C53, C54, C8: value 10uF -> GRM188R6YA106MA73D
- V1: now left out of the parts list
Connections:
- net BACK_EMF: now also SHUNT-2.1
- net BST: now also SHUNT+2.1
- net at MOSFET8.4, R66.2, R69.2: now also GATE_L2.1
- net at MOSFET7.4, R67.2, R68.2: now also GATE_H2.1
Other:
- note added: "Low ESR ceramic capacitors (10uF) placed near inverter leg"
- note removed: "Low ESR ceramic capacitors placed near inverter leg"

Commit message: added test points
Parts:
- removed GATE_H2, GATE_L2, SHUNT+2, SHUNT-2: TestPoint, TestPoint:TestPoint_Loop_D1.80mm_Drill1.0mm_Beaded, symbol Connector:TestPoint

Commit message: bom finished
Parts:
- C43, C53, C54, C8: value GRM188R6YA106MA73D -> 10u; MANUFACTURER (none) -> Murata Electronics; MPN (none) -> GRM188R6YA106MA73D; Supplier (none) -> Digikey
- MOSFET7, MOSFET8: value AON6512 -> NMOS; MANUFACTURER (none) -> Alpha & Omega Semiconductor Inc.; MPN (none) -> AON6512; Supplier (none) -> Digikey
- R66, R67: MANUFACTURER (none) -> YAGEO; MPN (none) -> RC0603FR-0722RL; Supplier (none) -> Digikey
- R68, R69: MANUFACTURER (none) -> YAGEO; MPN (none) -> RC0603FR-0710KL; Supplier (none) -> Digikey
- R70: MANUFACTURER (none) -> Stackpole Electronics Inc; MPN (none) -> CSSU2512FT5L00; Supplier (none) -> Digikey

Commit message: changed push buttons and zone clearances
Parts:
- C43, C53, C54, C8: value 10u -> GRM188R6YA106MA73D
Changed lines of the file:
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@@
 			)
 		)
-		(property "Value" "10u"
+		(property "Value" "GRM188R6YA106MA73D"
 			(at 205.994 49.53 0)
 			(effects
@@
 			)
 		)
-		(property "Value" "10u"
+		(property "Value" "GRM188R6YA106MA73D"
 			(at 246.38 44.4499 0)
 			(effects
@@
 			)
 		)
-		(property "Value" "10u"
+		(property "Value" "GRM188R6YA106MA73D"
 			(at 234.95 44.4499 0)
 			(effects
@@
 			)
 		)
-		(property "Value" "10u"
+		(property "Value" "GRM188R6YA106MA73D"
 			(at 229.362 49.784 0)
 			(effects

Commit message: reoriented parts
Parts:
- R66, R67: value 22 -> 0
Changed lines of the file:
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@@
 			)
 		)
-		(property "Value" "22"
+		(property "Value" "0"
 			(at 96.52 68.58 90)
 			(effects
@@
 			)
 		)
-		(property "Value" "22"
+		(property "Value" "0"
 			(at 95.25 140.97 90)
 			(effects
