File: flight-controller/Power Board.kicad_pcb (KiCad board)
At the start: 2 copper layers, 34 parts, among them J2 XT60-M, J3 Lipo JST, J4 MCU_Power, J5 XT60-M, J6 XT60-M, J7 Motor MCU 2, J8 Motor MCU 1, SW1 SW_Push, U1 AP64500SP-13, U3 BQ76920PW

Commit message: clean hierachy?
Parts:
- removed J4: MCU_Power, Connector_JST:JST_XH_S2B-XH-A_1x02_P2.50mm_Horizontal
- added A1: Arduino_Nano_ESP32, Module:Arduino_Nano, F.Cu at (183.1, 71.6)
- added Q2: NMOS, Package_SO:ONSemi_SO-8FL_488AA, F.Cu at (250.3, 106.1)
- moved J5 52.0 mm to (225.1, 84.4)
- moved R17 51.7 mm to (252.2, 96.2)
- moved J3 51.0 mm to (224.7, 90.8)
- moved R8 47.1 mm to (248.2, 96.2)
- moved C18 43.3 mm to (244.2, 93.7)
- moved J2 38.6 mm to (207.5, 84.4)
- moved C1 37.9 mm to (240.2, 88.7)
- moved C12 37.7 mm to (240.2, 93.7)
- moved C13 37.7 mm to (240.2, 96.2)
- moved C14 37.7 mm to (240.2, 98.7)
- moved C15 37.7 mm to (240.2, 101.3)
- moved J7 35.5 mm to (205.8, 90.8)
- moved J8 35.5 mm to (215.3, 90.8)
- moved SW1 34.1 mm to (223.3, 103.0)
- moved J6 33.5 mm to (242.6, 84.4)
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