File: flight-controller/Power Board.kicad_sch (KiCad schematic)
At the start: 48 parts, among them J1 MCU I2C, J2 XT60-M, J3 Lipo JST, J4 MCU_Power, J5 XT60-M, J6 XT60-M, J7 Motor MCU 2, J8 Motor MCU 1, Q2 NMOS, SW1 SW_Push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

Commit message: clean hierachy?
Parts:
- removed C1, C12, C16, C17, C19, C20, C21: 1u, Capacitor_SMD:C_0603_1608Metric, symbol Device:C
- removed C10: 10u, symbol Device:C
- removed C11: 2.7n, symbol Device:C
- removed C13, C14, C15: 0.1u, Capacitor_SMD:C_0603_1608Metric, symbol Device:C
- removed C18: 4.7u, Capacitor_SMD:C_0603_1608Metric, symbol Device:C
- removed C2: 10u, Capacitor_SMD:C_0603_1608Metric, symbol Device:C
- removed C6: 100n, symbol Device:C
- removed C7, C8, C9: 22u, symbol Device:C
- removed D1: PTVS18VZ1USK, Diode_SMD:Nexperia_DSN1608-2_1.6x0.8mm, symbol Diode:PTVS18VZ1USK
- removed J1: MCU I2C, symbol Connector:Conn_01x05_Socket
- removed J2, J5, J6: XT60-M, Connector_AMASS:AMASS_XT60IPW-M_1x03_P7.20mm_Horizontal, symbol XT60-M:XT60-M
- removed J3: Lipo JST, Connector_JST:JST_XH_S5B-XH-A_1x05_P2.50mm_Horizontal, symbol Connector:Conn_01x05_Socket
- removed J4: MCU_Power, Connector_JST:JST_XH_S2B-XH-A_1x02_P2.50mm_Horizontal, symbol Connector:Conn_01x02_Socket
- removed J7: Motor MCU 2, Connector_JST:JST_XH_S2B-XH-A_1x02_P2.50mm_Horizontal, symbol Connector:Conn_01x02_Socket
- removed J8: Motor MCU 1, Connector_JST:JST_XH_S2B-XH-A_1x02_P2.50mm_Horizontal, symbol Connector:Conn_01x02_Socket
- removed L2: 3.6u, symbol Device:L
- removed Q2: NMOS, symbol Simulation_SPICE:NMOS
- removed R1, R10, R11, R13, R16, R2, R9: 100, Resistor_SMD:R_0603_1608Metric, symbol Device:R
- removed R12: 100, symbol Device:R
- removed R17, R8: 10k, Resistor_SMD:R_0603_1608Metric, symbol Device:R
- removed R3: 115k, symbol Device:R
- removed R4: 22.1k, symbol Device:R
- removed R5: 200k, symbol Device:R
- removed R6: 15.8k, symbol Device:R
- removed R7: 1M, Resistor_SMD:R_0603_1608Metric, symbol Device:R
- removed Rsns1: 5m, Resistor_SMD:R_2512_6332Metric, symbol Device:R
- removed SW1: SW_Push, Button_Switch_THT:SW_PUSH_6mm, symbol Switch:SW_Push
- removed U1: AP64500SP-13, Package_SO:Diodes_SO-8EP, symbol 2026-04-01_21-43-48:AP64500SP-13
- removed U3: BQ76920PW, Package_SO:TSSOP-20_4.4x6.5mm_P0.65mm, symbol Battery_Management:BQ76920PW
Other:
- added sheet BMS (BMS.kicad_sch)
- added sheet Flight_Controller (FC.kicad_sch)
- note removed: "5V/5A buck converter"
- note removed: "BMS"
