File: flight-controller/BMS.kicad_sch (KiCad schematic)
At the start: 47 parts

Commit message: clean hierachy
Parts:
- removed J: Motor MCU 2, Connector_JST:JST_XH_S2B-XH-A_1x02_P2.50mm_Horizontal, symbol Connector:Conn_01x02_Socket
- removed J: Motor MCU 1, Connector_JST:JST_XH_S2B-XH-A_1x02_P2.50mm_Horizontal, symbol Connector:Conn_01x02_Socket
- removed J: XT60-M, Connector_AMASS:AMASS_XT60IPW-M_1x03_P7.20mm_Horizontal, symbol XT60-M:XT60-M
- Q2: renamed from Q; footprint Package_SO:ONSemi_SO-8FL_488AA -> Package_DFN_QFN:PQFN-8-EP_6x5mm_P1.27mm_Generic
- renumbered C to C1, C to C10, C to C11, C to C12, C to C13, C to C14, C to C15, C to C16, C to C17, C to C18, C to C19, C to C2, C to C20, C to C21, C to C6, C to C7, C to C8, C to C9, D to D1, J to J1, J to J3, J to J5, J to J6, L to L2, R to R1, R to R10, R to R11, R to R12, R to R13, R to R16, R to R17, R to R2, R to R3, R to R4, R to R5, R to R6, R to R7, R to R8, R to R9, Rsns to Rsns1, SW to SW1, U to U1, U to U3
Connections:
- net 5V: now reaches C8.1, L2.2, R3.2
- net Buck_In renamed 15V

Commit message: fc with esp
Connections:
- net 5V: now also C18.1, J1.1 (Pin_1)
- net GND: no longer C18.2
- net GND1: now also C18.2
- now unconnected: U3.8 (REGOUT)
- no-connect marks 0 -> 2

Commit message: sensors
Parts:
- removed C18: 4.7u, Capacitor_SMD:C_0603_1608Metric, symbol Device:C
- removed J1: MCU I2C, symbol Connector:Conn_01x05_Socket
Connections:
- net PWR_BTN: now reaches R17.1, R8.1, U3.6 (TS1)
- net SCL_BMS: now reaches U3.5 (SCL)
- net SDA_BMS: now reaches U3.4 (SDA)
- net INT_BMS: now reaches U3.20 (ALERT)
Other:
- moved on the sheet: C1, R17

Commit message: wa
Parts:
- removed J5, J6: XT60-M, Connector_AMASS:AMASS_XT60IPW-M_1x03_P7.20mm_Horizontal, symbol XT60-M:XT60-M
- added J10, J9: XT60PW-F, Connector_AMASS:AMASS_XT60PW-F_1x02_P7.20mm_Horizontal, symbol XT60PW-F:XT60PW-F
Connections:
- net 15V: now also J10.1 (P), J9.1 (P)
- net GND1: now also J10.2 (N), J9.2 (N)
- net SCL_BMS renamed SCL
- net SDA_BMS renamed SDA
- new net: J9.SH1 (SHIELD), J9.SH2 (SHIELD)
- new net: J10.SH1 (SHIELD), J10.SH2 (SHIELD)
- no-connect marks 2 -> 4
Other:
- moved on the sheet: D1

Commit message: cleaned up the layout
Parts:
- removed J10, J9: XT60PW-F, Connector_AMASS:AMASS_XT60PW-F_1x02_P7.20mm_Horizontal, symbol XT60PW-F:XT60PW-F
- removed J3: Lipo JST, Connector_JST:JST_XH_S5B-XH-A_1x05_P2.50mm_Horizontal, symbol Connector:Conn_01x05_Socket
Connections:
- net VC1: now reaches R10.1
- net VC3: now reaches R2.1
- net VC5: now reaches R16.1
- net VC0: now reaches R9.1
- net VC2: now reaches R13.1
- no-connect marks 4 -> 2
Other:
- moved on the sheet: SW1
