File: flight-controller/FC.kicad_sch (KiCad schematic)
At the start: 1 part, among them U2 ESP32-S3-MINI-1

Commit message: clean hierachy
Other:
- moved on the sheet: U2
Changed lines of the file:
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@@
 	(symbol
 		(lib_id "RF_Module:ESP32-S3-MINI-1")
-		(at 80.01 64.77 0)
+		(at 77.47 71.12 0)
 		(unit 1)
 		(body_style 1)
@@
 		(fields_autoplaced yes)
 		(property "Reference" "U2"
-			(at 82.1533 31.75 0)
+			(at 79.6133 38.1 0)
 			(show_name no)
 			(do_not_autoplace no)
@@
 		)
 		(property "Value" "ESP32-S3-MINI-1"
-			(at 82.1533 34.29 0)
+			(at 79.6133 40.64 0)
 			(show_name no)
 			(do_not_autoplace no)
@@
 		)
 		(property "Footprint" "RF_Module:ESP32-S2-MINI-1"
-			(at 95.25 93.98 0)
+			(at 92.71 100.33 0)
 			(hide yes)
 			(show_name no)
@@
 		)
 		(property "Datasheet" "https://www.espressif.com/sites/default/files/documentation/esp32-s3-mini-1_mini-1u_datasheet_en.pdf"
-			(at 80.01 24.13 0)
+			(at 77.47 30.48 0)
 			(hide yes)
 			(show_name no)
@@
 		)
 		(property "Description" "RF Module, ESP32-S3 SoC, Wi-Fi 802.11b/g/n, Bluetooth, BLE, 32-bit, 3.3V, SMD, onboard antenna"
-			(at 80.01 21.59 0)
+			(at 77.47 27.94 0)
 			(hide yes)
 			(show_name no)
@@
 		)
 		(instances
-			(project "Power Board"
+			(project "flight-controller"
 				(path "/e1d5dd76-ec41-4f53-aa0b-5d03fb935d99/ab31c291-e8bf-479a-b3ea-b25df21dfdbf"
 					(reference "U2")

Commit message: fc with esp
Parts:
- added C5: 10u, Capacitor_SMD:C_0603_1608Metric, symbol Device:C
- added J2: USB_B_Micro, Connector_USB:USB_Micro-B_Amphenol_10103594-0001LF_Horizontal, symbol Connector:USB_B_Micro
- added U4: NCP1117ST33T3G, Package_TO_SOT_SMD:SOT-223-3_TabPin2, symbol Regulator_Linear:NCP1117-3.3_SOT223
Connections:
- net GND1: now reaches U2.1 (GND), U2.2 (GND), U2.42 (GND), U2.43 (GND), U2.46 (GND), U2.47 (GND), U2.48 (GND), U2.49 (GND), U2.50 (GND), U2.51 (GND), U2.52 (GND), U2.53 (GND), U2.54 (GND), U2.55 (GND), U2.56 (GND), U2.57 (GND), U2.58 (GND), U2.59 (GND), U2.60 (GND), U2.61 (GND), U2.62 (GND), U2.63 (GND), U2.64 (GND), U2.65 (GND)
- net GND1: now also C5.2, J2.5 (GND), J2.SH (Shield), U4.1 (GND)
- net at U2.23 (USB_D-): now also J2.2 (D-)
- net at U2.24 (USB_D+): now also J2.3 (D+)
- net +3V3: now reaches U2.3 (3V3)
- net +3V3: now also C5.1, U4.2 (VO)
- new net 5V: J2.1 (VBUS), U4.3 (VI)
- no-connect marks 0 -> 1
Other:
- note added: "Power"
- moved on the sheet: U2

Commit message: sensors
Parts:
- added A1: ENS220S-BLGT, ENS220S-BLGT:XDCR_ENS220S-BLGT, symbol ENS220S-BLGT:ENS220S-BLGT
- added C18, C4: 0.1u, symbol Device:C
- added C22: 22u, symbol Device:C
- added C23, C24, C3: C, symbol Device:C
- added C25: 100n, symbol Device:C
- added R14, R15: 4.7k, symbol Device:R
- added SW2: SW_Push, symbol Switch:SW_Push
- added U6: NCP1117-1.8_SOT223, Package_TO_SOT_SMD:SOT-223-3_TabPin2, symbol Regulator_Linear:NCP1117-1.8_SOT223
- added U7: LSM6DSR, LGA_M6DSR_STM, symbol 2026-04-10_00-11-54:LSM6DSR
Connections:
- net +3V3: now also C22.1, C4.1, R14.1, R15.1
- net 5V: now also U6.3 (VI)
- net GND1: now also A1.3 (GND), A1.8 (GND__1), A1.9 (GND__2), C18.1, C22.2, C23.2, C24.2, C25.2, C3.2, C4.2, SW2.1, U6.1 (GND), U7.2 (SDX), U7.3 (SCX), U7.6 (GND), U7.7 (GND)
- net at J2.2 (D-), U2.23 (USB_D-): now also C23.1
- net at J2.3 (D+), U2.24 (USB_D+): now also C24.1
- net SCL_BMS: now reaches U2.10 (IO6)
- net SCL_BMS: now also A1.2 (SCL/SCLK), R14.2
- net SDA_BMS: now reaches U2.11 (IO7)
- net SDA_BMS: now also A1.4 (SDA/SDI), R15.2
- net INT_BMS: now reaches U2.12 (IO8)
- net INT_IMU: now reaches U2.13 (IO9)
- net INT_IMU: now also U7.4 (INT1)
- net CS: now reaches U2.14 (IO10)
- net CS: now also U7.12 (CS)
- net MOSI: now reaches U2.15 (IO11)
- net MOSI: now also U7.14 (SDA)
- net SCLK: now reaches U2.16 (IO12)
- net SCLK: now also U7.13 (SCL)
- net MISO: now reaches U2.17 (IO13)
- net MISO: now also U7.1 (SDO/SA0)
- net at U2.45 (EN): now also C18.2, SW2.2
- net PWR_BTN: now reaches U2.5 (IO1)
- new net +1V8: A1.10 (VDD), C25.1, C3.1, U6.2 (VO), U7.5 (VDD_IO), U7.8 (VDD)
- no-connect marks 1 -> 11
Other:
- note added: "Change to lower current rating ldo"
- moved on the sheet: C5, J2, U2, U4

Commit message: wa
Parts:
- added D2, D3: LED, symbol Device:LED
- SW2: footprint (none) -> Button_Switch_THT:SW_PUSH_6mm
Connections:
- net INT_BMS: now also U2.10 (IO6); no longer U2.12 (IO8)
- net INT_IMU: now also U2.11 (IO7); no longer U2.13 (IO9)
- net CS_MD1: now reaches U2.31 (IO35)
- net CS_MD2: now reaches U2.32 (IO36)
- net CS renamed CS_IMU
- net SCL_BMS renamed SCL
- net SCL: now also U2.12 (IO8); no longer U2.10 (IO6)
- net SDA_BMS renamed SDA
- net SDA: now also U2.13 (IO9); no longer U2.11 (IO7)
- no-connect marks 11 -> 14
Other:
- note added: "for low battery alert"
- note added: "for mcu power on/off"
- moved on the sheet: A1, C18, C25, R14, R15, SW2

Commit message: cleaned up the layout
Parts:
- removed A1: ENS220S-BLGT, ENS220S-BLGT:XDCR_ENS220S-BLGT, symbol ENS220S-BLGT:ENS220S-BLGT
- removed C23, C24, C3: C, symbol Device:C
- removed C25: 100n, symbol Device:C
- removed D3: LED, symbol Device:LED
- removed U6: NCP1117-1.8_SOT223, Package_TO_SOT_SMD:SOT-223-3_TabPin2, symbol Regulator_Linear:NCP1117-1.8_SOT223
- removed U7: LSM6DSR, LGA_M6DSR_STM, symbol 2026-04-10_00-11-54:LSM6DSR
- added D2: LED, LED_SMD:LED_0201_0603Metric, symbol Device:LED
- added Q1: NMOS, symbol Simulation_SPICE:NMOS
- added R20: 10k, symbol Device:R
- added R21, R22: 220, symbol Device:R
- D1: renamed from D2; footprint (none) -> LED_SMD:LED_0201_0603Metric
- SW2: value SW_Push -> RESET
Connections:
- net +3V3: now also U2.5 (IO1), Q1.1 (D)
- net GND1: now also R20.2, R21.2, R22.2
- net PWR_BTN: now also Q1.2 (G); no longer U2.5 (IO1)
- net at D1.1 (K): now also R21.1
- net LED_PWR: now reaches D1.2 (A)
- net LED_PWR: now also U2.21 (IO17)
- net LED_BMS: now reaches U2.22 (IO18)
- net LED_BMS: now also D2.2 (A)
- new net: Q1.3 (S), R20.1
- new net: D2.1 (K), R22.1
- no-connect marks 14 -> 25
Other:
- note added: "3V3 LDO"
- note added: "Add UART pins for GPS module?"
- note added: "ESP32"
- note added: "LED"
- note added: "Poweroff btn"
- note added: "add resistors and size fet Switch to a comparator"
- note removed: "Change to lower current rating ldo"
- note removed: "Power"
- moved on the sheet: C18, C22, C4, C5, D1, J2, R14, R15, SW2, U2, U4
