File: flight-controller/flight-controller.kicad_pcb (KiCad board)
At the start: 2 copper layers, 34 parts, among them J2 USB_B_Micro, J3 Lipo JST, J5 XT60-M, J6 XT60-M, J7 XT60-M, Q2 NMOS, SW1 SW_Push, U1 AP64500SP-13, U2 ESP32-S3-MINI-1, U3 BQ76920PW

Commit message: fc with esp
Parts:
- added C5: 10u, Capacitor_SMD:C_0603_1608Metric, F.Cu at (48.3, 74.1)
- added U4: NCP1117ST33T3G, Package_TO_SOT_SMD:SOT-223-3_TabPin2, F.Cu at (31.9, 77.0)
- moved J2 198.2 mm to (41.6, 76.7)
- moved U2 151.6 mm to (50.2, 61.8)
- moved C12 150.1 mm to (46.0, 109.8)
- moved C15 150.1 mm to (46.0, 117.4)
- moved C18 150.1 mm to (50.0, 109.8)
- moved C21 150.1 mm to (50.0, 117.4)
- moved D1 150.1 mm to (53.6, 119.8)
- moved J3 150.1 mm to (30.5, 106.9)
- moved R10 150.1 mm to (54.0, 117.4)
- moved R16 150.1 mm to (58.0, 109.8)
- moved R7 150.1 mm to (54.0, 109.8)
- moved SW1 150.1 mm to (29.0, 119.2)
- moved U1 150.1 mm to (48.0, 122.1)
- moved U3 150.1 mm to (64.7, 107.6)
- moved C1 150.1 mm to (46.0, 104.8)
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Connections:
- C18 pad 1: Net-(J1-Pin_1) -> 5V
- C18 pad 2: GND -> GND1
- J2 pad 1: unconnected-(J2-VBUS-Pad1) -> 5V
- J2 pad 2: unconnected-(J2-D--Pad2) -> Net-(J2-D-)
- J2 pad 3: unconnected-(J2-D+-Pad3) -> Net-(J2-D+)
- J2 pad 5: unconnected-(J2-GND-Pad5) -> GND1
- J2 pad SH: unconnected-(J2-Shield-PadSH) -> GND1
- U2 pad 1: Net-(U2-GND-Pad1) -> GND1
- U2 pad 2: Net-(U2-GND-Pad1) -> GND1
- U2 pad 23: unconnected-(U2-USB_D--Pad23) -> Net-(J2-D-)
- U2 pad 24: unconnected-(U2-USB_D+-Pad24) -> Net-(J2-D+)
- U2 pad 3: unconnected-(U2-3V3-Pad3) -> 3V3
- U2 pad 42: Net-(U2-GND-Pad1) -> GND1
- U2 pad 43: Net-(U2-GND-Pad1) -> GND1
- U2 pad 46: Net-(U2-GND-Pad1) -> GND1
- U2 pad 47: Net-(U2-GND-Pad1) -> GND1
- U2 pad 48: Net-(U2-GND-Pad1) -> GND1
- U2 pad 49: Net-(U2-GND-Pad1) -> GND1
- U2 pad 50: Net-(U2-GND-Pad1) -> GND1
- U2 pad 51: Net-(U2-GND-Pad1) -> GND1
- U2 pad 52: Net-(U2-GND-Pad1) -> GND1
- U2 pad 53: Net-(U2-GND-Pad1) -> GND1
- U2 pad 54: Net-(U2-GND-Pad1) -> GND1
- U2 pad 55: Net-(U2-GND-Pad1) -> GND1
- U2 pad 56: Net-(U2-GND-Pad1) -> GND1
- U2 pad 57: Net-(U2-GND-Pad1) -> GND1
- U2 pad 58: Net-(U2-GND-Pad1) -> GND1
- U2 pad 59: Net-(U2-GND-Pad1) -> GND1
- U2 pad 60: Net-(U2-GND-Pad1) -> GND1
- U2 pad 61: Net-(U2-GND-Pad1) -> GND1
- U2 pad 62: Net-(U2-GND-Pad1) -> GND1
- U2 pad 63: Net-(U2-GND-Pad1) -> GND1
- U2 pad 64: Net-(U2-GND-Pad1) -> GND1
- U2 pad 65: Net-(U2-GND-Pad1) -> GND1
- U3 pad 8: Net-(J1-Pin_1) -> unconnected-(U3-REGOUT-Pad8)

Commit message: sensors
Parts:
- added U5: LSM6DSM, Package_LGA:LGA-14_3x2.5mm_P0.5mm_LayoutBorder3x4y, F.Cu at (97.9, 127.8)
- moved C5 75.2 mm to (97.3, 131.1)
- moved C14 72.2 mm to (95.0, 167.9)
- moved C17 72.2 mm to (99.0, 160.3)
- moved C2 72.2 mm to (95.0, 160.3)
- moved C20 72.2 mm to (99.0, 167.9)
- moved Q2 72.2 mm to (113.1, 173.0)
- moved R13 72.2 mm to (107.0, 160.3)
- moved C12 72.2 mm to (95.0, 162.8)
- moved C15 72.2 mm to (95.0, 170.4)
- moved C18 72.2 mm to (99.0, 162.8)
- moved C21 72.2 mm to (99.0, 170.4)
- moved D1 72.2 mm to (102.6, 172.8)
- moved J2 72.2 mm to (90.6, 129.7)
- moved J3 72.2 mm to (79.5, 159.9)
- moved J5 72.2 mm to (81.2, 153.5)
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
Commit message: wa
Parts:
- removed C18: 4.7u, Capacitor_SMD:C_0603_1608Metric
- removed J5, J6, J7: XT60-M, Connector_AMASS:AMASS_XT60IPW-M_1x03_P7.20mm_Horizontal
- removed U5: LSM6DSM, Package_LGA:LGA-14_3x2.5mm_P0.5mm_LayoutBorder3x4y
- added J1: Motor_Driver_1, Connector_JST:JST_XH_S4B-XH-A_1x04_P2.50mm_Horizontal, F.Cu at (89.9, 92.3)
- added J10: XT60PW-F, Connector_AMASS:AMASS_XT60PW-F_1x02_P7.20mm_Horizontal, F.Cu at (116.4, 62.4)
- added J4: Motor_Driver_2, Connector_JST:JST_XH_S4B-XH-A_1x04_P2.50mm_Horizontal, F.Cu at (89.9, 105.9)
- added J8: XT60PW-F, Connector_AMASS:AMASS_XT60PW-F_1x02_P7.20mm_Horizontal, F.Cu at (113.3, 105.3)
- added J9: XT60PW-F, Connector_AMASS:AMASS_XT60PW-F_1x02_P7.20mm_Horizontal, F.Cu at (98.8, 62.4)
- added SW2: SW_Push, Button_Switch_THT:SW_PUSH_6mm, F.Cu at (49.9, 84.3)
- added U6: NCP1117-1.8_SOT223, Package_TO_SOT_SMD:SOT-223-3_TabPin2, F.Cu at (42.9, 94.8)
- moved SW1 111.9 mm to (117.5, 67.5)
- moved R10 98.9 mm to (96.5, 71.7)
- moved R9 98.9 mm to (96.5, 69.2)
- moved R8 98.9 mm to (96.5, 66.7)
- moved C20 96.4 mm to (92.5, 71.7)
- moved C21 96.4 mm to (92.5, 74.2)
- moved C19 96.4 mm to (92.5, 69.2)
- moved C17 93.9 mm to (92.5, 66.7)
- moved J3 93.9 mm to (102.0, 68.8)
- moved U1 93.7 mm to (110.9, 82.5)
- moved C12 91.4 mm to (88.5, 71.7)
- moved C14 91.4 mm to (88.5, 76.7)
- moved C15 91.4 mm to (88.5, 79.3)
- moved C2 91.4 mm to (88.5, 69.2)
- moved C1 91.4 mm to (88.5, 66.7)
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Connections:
- net /BMS/Buck_In renamed /BMS/15V
- R17 pad 1: Net-(U3-TS1) -> /BMS/PWR_BTN
- R8 pad 1: Net-(U3-TS1) -> /BMS/PWR_BTN
- U2 pad 10: unconnected-(U2-IO6-Pad10) -> /BMS/INT_BMS
- U2 pad 11: unconnected-(U2-IO7-Pad11) -> /Flight_Controller/INT_IMU
- U2 pad 12: unconnected-(U2-IO8-Pad12) -> /Flight_Controller/SCL
- U2 pad 13: unconnected-(U2-IO9-Pad13) -> /Flight_Controller/SDA
- U2 pad 14: unconnected-(U2-IO10-Pad14) -> /Flight_Controller/CS_IMU
- U2 pad 15: unconnected-(U2-IO11-Pad15) -> /Flight_Controller/MOSI
- U2 pad 16: unconnected-(U2-IO12-Pad16) -> /Flight_Controller/SCLK
- U2 pad 17: unconnected-(U2-IO13-Pad17) -> /Flight_Controller/MISO
- U2 pad 31: unconnected-(U2-IO35-Pad31) -> /Flight_Controller/CS_MD1
- U2 pad 32: unconnected-(U2-IO36-Pad32) -> /Flight_Controller/CS_MD2
- U2 pad 45: unconnected-(U2-EN-Pad45) -> Net-(U2-EN)
- U2 pad 5: unconnected-(U2-IO1-Pad5) -> /BMS/PWR_BTN
- U3 pad 20: Net-(J1-Pin_4) -> /BMS/INT_BMS
- U3 pad 4: Net-(J1-Pin_3) -> /Flight_Controller/SDA
- U3 pad 5: Net-(J1-Pin_2) -> /Flight_Controller/SCL
- U3 pad 6: Net-(U3-TS1) -> /BMS/PWR_BTN

Commit message: cleaned up the layout
Parts:
- added U5: LIS2MDL, Package_LGA:LGA-12_2x2mm_P0.5mm, F.Cu at (56.4, 114.9)
- J1: value Motor_Driver_1 -> MD1_SPI
- J10: value XT60PW-F -> MD2_15V
- J4: value Motor_Driver_2 -> MD2_SPI
- J9: value XT60PW-F -> MD1_15V
- SW2: value SW_Push -> RESET
- moved J8 92.2 mm to (46.4, 41.9)
- moved J1 68.5 mm to (37.5, 48.3)
- moved J4 68.5 mm to (37.5, 61.8)
- moved J10 40.5 mm to (81.5, 41.9)
- moved J9 40.5 mm to (63.9, 41.9)
- moved Rsns1 36.9 mm to (86.8, 100.9)
- moved SW1 30.5 mm to (96.5, 89.7)
- moved U3 30.5 mm to (99.2, 100.2)
- moved J2 28.4 mm to (48.6, 122.8)
- moved SW2 28.4 mm to (45.9, 112.4)
- moved U2 28.4 mm to (57.2, 99.3)
- moved U4 28.4 mm to (38.9, 114.6)
- moved U6 28.4 mm to (38.9, 122.9)
- moved C5 24.6 mm to (56.4, 111.6)
- moved Q2 20.4 mm to (86.5, 95.1)
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