File: flight-controller/flight-controller.kicad_sch (KiCad schematic)
At the start: 1 part, among them J7 XT60-M

Commit message: fc with esp
Other:
- sheet Flight_Controller ports: added 5V; removed none
Changed lines of the file:
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@@
+	(wire
+		(pts
+			(xy 160.02 50.8) (xy 165.1 50.8)
+		)
+		(stroke
+			(width 0)
+			(type default)
+		)
+	)
 	(wire
 		(pts
@@
 	)
 	(sheet
-		(at 114.3 86.36)
-		(size 45.72 33.02)
+		(at 165.1 44.45)
+		(size 45.72 31.75)
 		(exclude_from_sim no)
 		(in_bom yes)
@@
 		)
 		(property "Sheetname" "Flight_Controller"
-			(at 114.3 85.6484 0)
+			(at 165.1 43.7384 0)
 			(show_name no)
 			(do_not_autoplace no)
@@
 		)
 		(property "Sheetfile" "FC.kicad_sch"
-			(at 114.3 119.9646 0)
+			(at 165.1 76.7846 0)
 			(show_name no)
 			(do_not_autoplace no)
@@
 			)
 		)
+		(pin "5V" input
+			(at 165.1 50.8 180)
+			(effects
+				(font
+					(size 1.27 1.27)
+				)
+				(justify left)
+			)
+		)

Commit message: sensors
Other:
- sheet BMS ports: added INT_BMS, PWR_BTN, SCL_BMS, SDA_BMS; removed none
- sheet Flight_Controller ports: added INT_BMS, PWR_BTN, SCL_BMS, SDA_BMS; removed none
Changed lines of the file:
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@@
 	(wire
 		(pts
-			(xy 160.02 50.8) (xy 165.1 50.8)
+			(xy 152.4 53.34) (xy 165.1 53.34)
 		)
 		(stroke
@@
 	(wire
 		(pts
-			(xy 67.31 50.8) (xy 114.3 50.8)
+			(xy 152.4 63.5) (xy 165.1 63.5)
+		)
+		(stroke
+			(width 0)
+			(type default)
+		)
+	)
+	(wire
+		(pts
+			(xy 152.4 50.8) (xy 165.1 50.8)
+		)
+		(stroke
+			(width 0)
+			(type default)
+		)
+	)
+	(wire
+		(pts
+			(xy 152.4 58.42) (xy 165.1 58.42)
+		)
+		(stroke
+			(width 0)
+			(type default)
+		)
+	)
+	(wire
+		(pts
+			(xy 67.31 50.8) (xy 106.68 50.8)
+		)
+		(stroke
+			(width 0)
+			(type default)
+		)
+	)
+	(wire
+		(pts
+			(xy 152.4 60.96) (xy 165.1 60.96)
 		)
 		(stroke
@@
 	)
 	(sheet
-		(at 114.3 44.45)
+		(at 106.68 44.45)
 		(size 45.72 31.75)
 		(exclude_from_sim no)
@@
 		)
 		(property "Sheetname" "BMS"
-			(at 114.3 43.7384 0)
+			(at 106.68 43.7384 0)
 			(show_name no)
 			(do_not_autoplace no)
@@
 		)
 		(property "Sheetfile" "BMS.kicad_sch"
-			(at 114.3 76.7846 0)
+			(at 106.68 76.7846 0)
 			(show_name no)
 			(do_not_autoplace no)
@@
 		)
 		(pin "5V" output
-			(at 160.02 50.8 0)
+			(at 152.4 50.8 0)
 			(effects
 				(font
@@
 		)
 		(pin "15V" input
-			(at 114.3 50.8 180)
+			(at 106.68 50.8 180)
 			(effects
 				(font
@@
 				)
 				(justify left)
+			)
+		)
+		(pin "SCL_BMS" input
+			(at 152.4 58.42 0)
+			(effects
+				(font
+					(size 1.27 1.27)
+				)
+				(justify right)
+			)
+		)
+		(pin "SDA_BMS" bidirectional
+			(at 152.4 60.96 0)
+			(effects
+				(font
+					(size 1.27 1.27)
+				)
+				(justify right)
+			)
+		)
+		(pin "PWR_BTN" output
+			(at 152.4 53.34 0)
+			(effects
+				(font
+					(size 1.27 1.27)
+				)
+				(justify right)
+			)
+		)
+		(pin "INT_BMS" output
+			(at 152.4 63.5 0)
+			(effects
+				(font
+					(size 1.27 1.27)
+				)
+				(justify right)
 			)
 		)
@@
 			(effects
 				(font
+					(size 1.27 1.27)
+				)
+				(justify left)
+			)
+		)
+		(pin "PWR_BTN" input
+			(at 165.1 53.34 180)
+			(effects
+				(font
+					(size 1.27 1.27)
+				)
+				(justify left)
+			)
+		)
+		(pin "INT_BMS" input
+			(at 165.1 63.5 180)
+			(effects
+				(font
+					(size 1.27 1.27)
+				)
+				(justify left)
+			)
+		)
+		(pin "SDA_BMS" bidirectional
+			(at 165.1 60.96 180)
+			(effects
+				(font
+					(size 1.27 1.27)
+				)
+				(justify left)
+			)
+		)
+		(pin "SCL_BMS" output
+			(at 165.1 58.42 180)
+			(effects
+				(font

Commit message: wa
Parts:
- removed J7: XT60-M, Connector_AMASS:AMASS_XT60IPW-M_1x03_P7.20mm_Horizontal, symbol XT60-M:XT60-M
- added J1: Motor_Driver_1, Connector_JST:JST_XH_S4B-XH-A_1x04_P2.50mm_Horizontal, symbol Connector:Conn_01x04_Socket
- added J4: Motor_Driver_2, Connector_JST:JST_XH_S4B-XH-A_1x04_P2.50mm_Horizontal, symbol Connector:Conn_01x04_Socket
- added J5: MD1_5V, B2B-PH-SM4-TB:JST_B2B-PH-SM4-TB, symbol B2B-PH-SM4-TB:B2B-PH-SM4-TB
- added J6: MD2_5V, B2B-PH-SM4-TB:JST_B2B-PH-SM4-TB, symbol B2B-PH-SM4-TB:B2B-PH-SM4-TB
- added J8: XT60PW-F, Connector_AMASS:AMASS_XT60PW-F_1x02_P7.20mm_Horizontal, symbol XT60PW-F:XT60PW-F
Connections:
- net BMS/15V: now also J8.1 (P)
- net BMS/5V: now also J5.1, J6.1
- net GND: now also J8.2 (N)
- new net: J8.SH1 (SHIELD), J8.SH2 (SHIELD)
- new net BMS/GND1: J5.2, J6.2
- new net Flight_Controller/CS_MD1: J1.3 (Pin_3)
- new net Flight_Controller/CS_MD2: J4.3 (Pin_3)
- new net Flight_Controller/MISO: J1.1 (Pin_1), J4.1 (Pin_1)
- new net Flight_Controller/MOSI: J1.4 (Pin_4), J4.4 (Pin_4)
- new net Flight_Controller/SCLK: J1.2 (Pin_2), J4.2 (Pin_2)
- no-connect marks 0 -> 1
Other:
- sheet BMS ports: added GND, GND1, SCL, SDA; removed SCL_BMS, SDA_BMS
- sheet Flight_Controller ports: added CS_MD1, CS_MD2, GND1, MISO, MOSI, SCL, SCLK, SDA; removed SCL_BMS, SDA_BMS
- note added: "5V Power Connection"

Commit message: cleaned up the layout
Parts:
- added J10: MD2_15V, Connector_AMASS:AMASS_XT60PW-F_1x02_P7.20mm_Horizontal, symbol XT60PW-F:XT60PW-F
- added J3: Lipo_Cell_Voltages, Connector_JST:JST_XH_S5B-XH-A_1x05_P2.50mm_Horizontal, symbol Connector:Conn_01x05_Socket
- added J9: MD1_15V, Connector_AMASS:AMASS_XT60PW-F_1x02_P7.20mm_Horizontal, symbol XT60PW-F:XT60PW-F
- J1: value Motor_Driver_1 -> MD1_SPI
- J4: value Motor_Driver_2 -> MD2_SPI
- J8: value XT60PW-F -> Lipo
Connections:
- net BMS/GND1: now also J10.2 (N), J9.2 (N)
- new net: J10.SH1 (SHIELD), J10.SH2 (SHIELD)
- new net: J9.SH1 (SHIELD), J9.SH2 (SHIELD)
- new net BMS/MD_15V: J10.1 (P), J9.1 (P)
- new net BMS/VC0: J3.1 (Pin_1)
- new net BMS/VC1: J3.2 (Pin_2)
- new net BMS/VC2: J3.3 (Pin_3)
- new net BMS/VC3: J3.4 (Pin_4)
- new net BMS/VC5: J3.5 (Pin_5)
- no-connect marks 1 -> 3
Other:
- sheet Flight_Controller renamed ESP32
- added sheet Sensors (Sensors.kicad_sch)
- sheet BMS ports: added MD_15V, VC0, VC1, VC2, VC3, VC5; removed none
- sheet ESP32 ports: added CS_IMU, INT_IMU; removed none
- note added: "15V Power Connection"
- note added: "Do not daisy chain!!"
- note added: "Motor Driver SPI"
- moved on the sheet: J1, J4, J5, J6, J8
